File: Crossi_Shield/CAN_Controller.kicad_sch (KiCad schematic)
At the start: 46 parts, among them IC2 TCAN1048AVDMTRQ1, IC3 TCAN1048AVDMTRQ1, IC4 TCAN1048AVDMTRQ1

Commit message: DSUB stecker neu
Connections:
- net at H3.20 (RXCAN), IC3.4 (RXD1): now also JP3.1 (A)
- net at H5.20 (RXCAN), IC4.4 (RXD1): now also JP5.1 (A)
- net at H1.20 (RXCAN), IC2.4 (RXD1): now also JP2.1 (A)
Changed lines of the file:
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@@
   (junction (at 121.92 168.91) (diameter 0) (color 0 0 0 0)
   )
+  (junction (at 176.53 82.55) (diameter 0) (color 0 0 0 0)
+  )
   (junction (at 182.88 246.38) (diameter 0) (color 0 0 0 0)
   )
@@
   (junction (at 154.94 264.16) (diameter 0) (color 0 0 0 0)
   )
+  (junction (at 462.28 86.36) (diameter 0) (color 0 0 0 0)
+  )
   (junction (at 243.84 82.55) (diameter 0) (color 0 0 0 0)
   )
@@
   )
   (junction (at 73.66 262.89) (diameter 0) (color 0 0 0 0)
+  )
+  (junction (at 175.26 254) (diameter 0) (color 0 0 0 0)
   )
   (junction (at 46.99 340.36) (diameter 0) (color 0 0 0 0)
@@
     (stroke (width 0) (type default))
   )
+  (wire (pts (xy 175.26 254) (xy 66.04 254))
+    (stroke (width 0) (type default))
+  )
   (wire (pts (xy 199.39 248.92) (xy 194.31 248.92))
     (stroke (width 0) (type default))
@@
     (stroke (width 0) (type default))
   )
+  (wire (pts (xy 176.53 82.55) (xy 67.31 82.55))
+    (stroke (width 0) (type default))
+  )
   (wire (pts (xy 99.06 336.55) (xy 93.98 336.55))
     (stroke (width 0) (type default))
@@
     (stroke (width 0) (type default))
   )
+  (wire (pts (xy 175.26 240.03) (xy 175.26 254))
+    (stroke (width 0) (type default))
+  )
   (wire (pts (xy 182.88 259.08) (xy 199.39 259.08))
     (stroke (width 0) (type default))
@@
     (stroke (width 0) (type default))
   )
+  (wire (pts (xy 462.28 86.36) (xy 353.06 86.36))
+    (stroke (width 0) (type default))
+  )
   (wire (pts (xy 140.97 90.17) (xy 176.53 90.17))
     (stroke (width 0) (type default))
@@
     (stroke (width 0) (type default))
   )
-  (wire (pts (xy 486.41 86.36) (xy 353.06 86.36))
+  (wire (pts (xy 486.41 86.36) (xy 462.28 86.36))
     (stroke (width 0) (type default))
   )
@@
     (stroke (width 0) (type default))
   )
-  (wire (pts (xy 175.26 240.03) (xy 175.26 252.73))
-    (stroke (width 0) (type default))
-  )
   (wire (pts (xy 243.84 105.41) (xy 243.84 107.95))
     (stroke (width 0) (type default))
@@
     (stroke (width 0) (type default))
   )
-  (wire (pts (xy 176.53 68.58) (xy 176.53 81.28))
+  (wire (pts (xy 176.53 68.58) (xy 176.53 82.55))
     (stroke (width 0) (type default))
   )
@@
     (stroke (width 0) (type default))
   )
-  (wire (pts (xy 462.28 72.39) (xy 462.28 85.09))
+  (wire (pts (xy 462.28 72.39) (xy 462.28 86.36))
     (stroke (width 0) (type default))
   )
@@
     (stroke (width 0) (type default))
   )
-  (wire (pts (xy 200.66 82.55) (xy 67.31 82.55))
+  (wire (pts (xy 200.66 82.55) (xy 176.53 82.55))
     (stroke (width 0) (type default))
   )
@@
     (stroke (width 0) (type default))
   )
-  (wire (pts (xy 199.39 254) (xy 66.04 254))
-    (stroke (width 0) (type default))
-  )
+  (wire (pts (xy 199.39 254) (xy 175.26 254))
+    (stroke (width 0) (type default))
+  )

Commit message: Fast fertig gerouted
Connections:
- net CAN0_H: now also R15.2
- net CAN0_L: now also JP2.1 (A)
- net CAN1_H: now also R14.1
- net CAN1_L: now also JP1.2 (B)
- net CAN2_H: now also R18.2
- net CAN2_L: now also JP3.1 (A)
- net CAN3_H: now also R19.1
- net CAN3_L: now also JP4.2 (B)
- net CAN4_H: now also R22.2
- net CAN4_L: now also JP5.1 (A)
- net at H3.19 (TXCAN), IC3.1 (TXD1): no longer R18.2
- net at H3.20 (RXCAN), IC3.4 (RXD1): no longer JP3.1 (A)
- net at H4.19 (TXCAN), IC3.6 (TXD2): no longer R19.1
- net at H4.20 (RXCAN), IC3.7 (RXD2): no longer JP4.2 (B)
- net at H2.19 (TXCAN), IC2.6 (TXD2): no longer R14.1
- net at H2.20 (RXCAN), IC2.7 (RXD2): no longer JP1.2 (B)
- net at H5.19 (TXCAN), IC4.1 (TXD1): no longer R22.2
- net at H5.20 (RXCAN), IC4.4 (RXD1): no longer JP5.1 (A)
- net at H1.19 (TXCAN), IC2.1 (TXD1): no longer R15.2
- net at H1.20 (RXCAN), IC2.4 (RXD1): no longer JP2.1 (A)
Other:
- moved on the sheet: JP1, JP2, JP3, JP4, JP5, R14, R15, R18, R19, R22
