File: Crossi_Shield/Versorgung.kicad_sch (KiCad schematic)
At the start: 25 parts, among them IC1 TPS54540DDAR

Commit message: DSUB stecker neu
Parts:
- R1: footprint Resistor_SMD:R_1218_3246Metric_Pad1.22x4.75mm_HandSolder -> Resistor_SMD:R_0805_2012Metric_Pad1.20x1.40mm_HandSolder
Changed lines of the file:
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@@
       (effects (font (size 1.27 1.27)) (justify left))
     )
-    (property "Footprint" "Resistor_SMD:R_1218_3246Metric_Pad1.22x4.75mm_HandSolder" (at 93.472 53.34 90)
+    (property "Footprint" "Resistor_SMD:R_0805_2012Metric_Pad1.20x1.40mm_HandSolder" (at 93.472 53.34 90)
       (effects (font (size 1.27 1.27)) hide)
     )

Commit message: Fast fertig gerouted
Connections:
- net BOOT: now reaches C6.2, D1.1, IC1.8 (SW), L1.1
Changed lines of the file:
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@@
     (effects (font (size 1.27 1.27) bold) (justify right bottom))
+  )
+  (label "BOOT" (at 146.05 40.64 0) (fields_autoplaced)
+    (effects (font (size 1.27 1.27)) (justify left bottom))
   )
   (hierarchical_label "5V" (shape input) (at 276.86 40.64 0) (fields_autoplaced)
